File: led-dimmer/led-dimmer.kicad_pcb (KiCad board)
At the start: 2 copper layers, 27.6 x 30.5 mm, 24 parts, among them J1 Conn_01x02_Pin, J2 Conn_01x02_Pin, Q1 IRLML6344, U1 NE555P

Commit message: Removed vias in pad from LED Dimmer PCB
Routing:
- net LED_PWM: track 14.1 -> 14.8 mm, vias 1 -> 2
- net GND: vias 37 -> 44
Other:
- board text added: "LED Dimmer Rev. 1.2"
- board text removed: "LED Dimmer Rev. 1.1"
Changed lines of the file:
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@@
 	(title_block
 		(title "LED Dimmer PCB")
-		(date "2026-08-15")
-		(rev "1.1")
+		(date "2026-09-09")
+		(rev "1.2")
 	)
 	(layers
@@
 		(layer "Edge.Cuts")
 	)
-	(gr_text "LED Dimmer\nRev. 1.1"
+	(gr_text "LED Dimmer\nRev. 1.2"
 		(at 75 124.6 90)
 		(layer "F.SilkS")
@@
 	)
 	(segment
+		(start 91.125001 112.225)
+		(end 89.5 112.225)
+		(width 0.5)
+		(layer "F.Cu")
+		(net "Net-(U1-OUT)")
+	)
+	(via
+		(at 89.5 112.225)
+		(size 0.6)
+		(drill 0.3)
+		(layers "F.Cu" "B.Cu")
+		(net "Net-(U1-OUT)")
+	)
+	(segment
+		(start 86.83 112.225)
+		(end 83.855 109.25)
+		(width 0.5)
+		(layer "B.Cu")
+		(net "Net-(U1-OUT)")
+	)
+	(segment
+		(start 89.5 112.225)
+		(end 86.83 112.225)
+		(width 0.5)
+		(layer "B.Cu")
+		(net "Net-(U1-OUT)")
+	)
+	(segment
 		(start 86.395 107.455)
 		(end 86.4 107.45)
@@
 	)
 	(via
+		(at 89 101.5)
+		(size 0.6)
+		(drill 0.3)
+		(layers "F.Cu" "B.Cu")
+		(free yes)
+		(net "GND")
+	)
+	(via
+		(at 78 113)
+		(size 0.6)
+		(drill 0.3)
+		(layers "F.Cu" "B.Cu")
+		(free yes)
+		(net "GND")
+	)
+	(via
 		(at 95.5 107.5)
 		(size 0.6)
@@
 	)
 	(via
+		(at 92 103.5)
+		(size 0.6)
+		(drill 0.3)
+		(layers "F.Cu" "B.Cu")
+		(free yes)
+		(net "GND")
+	)
+	(via
+		(at 92 101.5)
+		(size 0.6)
+		(drill 0.3)
+		(layers "F.Cu" "B.Cu")
+		(free yes)
+		(net "GND")
+	)
+	(via
+		(at 77 113)
+		(size 0.6)
+		(drill 0.3)
+		(layers "F.Cu" "B.Cu")
+		(free yes)
+		(net "GND")
+	)
+	(via
 		(at 80 114.5)
 		(size 0.6)
@@
 	)
 	(via
-		(at 79.05 115.325)
+		(at 92 102.5)
+		(size 0.6)
+		(drill 0.3)
+		(layers "F.Cu" "B.Cu")
+		(free yes)
+		(net "GND")
+	)
+	(via
+		(at 91 107.5)
 		(size 0.6)
 		(drill 0.3)
 		(layers "F.Cu" "B.Cu")
+		(free yes)
 		(net "GND")
 	)
@@
 	)
 	(via
-		(at 91.267499 108.8375)
+		(at 92.5 113.5)
 		(size 0.6)
 		(drill 0.3)
 		(layers "F.Cu" "B.Cu")
+		(free yes)
 		(net "GND")
 	)
 	(via
-		(at 92.5 113.5)
+		(at 76 113)
 		(size 0.6)
 		(drill 0.3)
@@
 	)
 	(via
+		(at 90 107.5)
+		(size 0.6)
+		(drill 0.3)
+		(layers "F.Cu" "B.Cu")
+		(free yes)
+		(net "GND")
+	)
+	(via
 		(at 90.5 113.5)
 		(size 0.6)
@@
 	)
 	(via
-		(at 78 114.5)
+		(at 92.25 108.75)
 		(size 0.6)
 		(drill 0.3)
@@
 	)
 	(via
-		(at 74.919999 110.967621)
+		(at 91 101.5)
 		(size 0.6)
 		(drill 0.3)
@@
 	)
 	(via
-		(at 82 106.5)
+		(at 78 114.5)
 		(size 0.6)
 		(drill 0.3)
@@
 	)
 	(via
-		(at 94.5 107.5)
+		(at 82 106.5)
 		(size 0.6)
 		(drill 0.3)
@@
 	)
 	(via
-		(at 87 106.5)
+		(at 94.5 107.5)
 		(size 0.6)
 		(drill 0.3)
@@
 	)
 	(via
-		(at 94.675 110.4875)
+		(at 75 112)
 		(size 0.6)
 		(drill 0.3)
 		(layers "F.Cu" "B.Cu")
+		(free yes)
 		(net "GND")
 	)
 	(via
-		(at 74.92 112.967623)
+		(at 87 106.5)
 		(size 0.6)
 		(drill 0.3)
@@
 	)
 	(via
-		(at 95.5 110.5)
+		(at 90 101.5)
 		(size 0.6)
 		(drill 0.3)
@@
 	)
 	(via
-		(at 79 114.5)
+		(at 78 112)
 		(size 0.6)
 		(drill 0.3)
@@
 	)
 	(via
-		(at 87.95 107.45)
+		(at 95.5 110.5)
 		(size 0.6)
 		(drill 0.3)
 		(layers "F.Cu" "B.Cu")
+		(free yes)
 		(net "GND")
 	)
 	(via
-		(at 95.5 109.5)
+		(at 79 114.5)
 		(size 0.6)
 		(drill 0.3)
@@
 	)
 	(via
-		(at 76.919997 112.967622)
+		(at 95.5 109.5)
 		(size 0.6)
 		(drill 0.3)
@@
 	)
 	(via
-		(at 95.5 108.5)
+		(at 78 111)
 		(size 0.6)
 		(drill 0.3)
@@
 	)
 	(via
-		(at 94.5 113.5)
+		(at 92 104.5)
 		(size 0.6)
 		(drill 0.3)
@@
 	)
 	(via
-		(at 84 107.5)
+		(at 95.5 108.5)
 		(size 0.6)
 		(drill 0.3)
@@
 	)
 	(via
-		(at 91.5 113.5)
+		(at 94.5 113.5)
 		(size 0.6)
 		(drill 0.3)
@@
 	)
 	(via
-		(at 82.875 107.45)
+		(at 75 113)
 		(size 0.6)
 		(drill 0.3)
 		(layers "F.Cu" "B.Cu")
+		(free yes)
 		(net "GND")
 	)
 	(via
-		(at 89 107.5)
+		(at 84 107.5)
 		(size 0.6)
 		(drill 0.3)
@@
 	)
 	(via
-		(at 75.919999 112.96762)
+		(at 91.5 113.5)
 		(size 0.6)
 		(drill 0.3)
@@
 	)
 	(via
-		(at 74.919997 111.967622)
+		(at 75 111)
 		(size 0.6)
 		(drill 0.3)
@@
 	)
 	(via
-		(at 78 116.5)
+		(at 89 107.5)
 		(size 0.6)
 		(drill 0.3)
@@
 	)
 	(via
-		(at 90.5 107.5)
+		(at 78 116.5)
 		(size 0.6)
 		(drill 0.3)
@@
 	)
 	(segment
+		(start 79.055 116.87)
+		(end 79.05 116.875)
+		(width 0.2)
+		(layer "F.Cu")
+		(net "Net-(U1-CONT)")
+	)
+	(segment
+		(start 81.315 116.87)
+		(end 79.055 116.87)
+		(width 0.5)
+		(layer "F.Cu")
+		(net "Net-(U1-CONT)")
+	)
+	(segment
 		(start 86.6125 101.572499)
 		(end 80.927499 101.572499)
@@
 	)
 	(segment
-		(start 93.725 108.6125)
+		(start 92.436274 107.323774)
+		(end 92.93125 107.81875)
+		(width 1)
+		(layer "F.Cu")
+		(net "LED_PWM")
+	)
+	(segment
+		(start 93.7125 108.6)
 		(end 93.725 108.6)
 		(width 1)
@@
 		(net "LED_PWM")
 	)
+	(segment
+		(start 92.93125 107.81875)
+		(end 93.7125 108.6)
+		(width 1)
+		(layer "F.Cu")
+		(net "LED_PWM")
+	)
 	(via
-		(at 93.725 108.6125)
+		(at 92.93125 107.81875)
+		(size 0.6)
+		(drill 0.3)
+		(layers "F.Cu" "B.Cu")
+		(net "LED_PWM")
+	)
+	(via
+		(at 92.436274 107.323774)
 		(size 0.6)
 		(drill 0.3)
@@
 	)
 	(segment
-		(start 90.6125 105.5)
-		(end 93.725 108.6125)
+		(start 92.93125 107.81875)
+		(end 90.6125 105.5)
 		(width 1)
 		(layer "B.Cu")
@@
 		(net "LED_PWM")
 	)
-	(segment
-		(start 79.055 116.87)
-		(end 79.05 116.875)
-		(width 0.2)
-		(layer "F.Cu")
-		(net "Net-(U1-CONT)")
-	)
-	(segment
-		(start 81.315 116.87)
-		(end 79.055 116.87)
-		(width 0.5)
-		(layer "F.Cu")
-		(net "Net-(U1-CONT)")
-	)
-	(via
-		(at 91.125002 112.225)
-		(size 0.6)
-		(drill 0.3)
-		(layers "F.Cu" "B.Cu")
-		(net "Net-(U1-OUT)")
-	)
-	(segment
-		(start 86.83 112.225)
-		(end 83.855 109.25)
-		(width 0.5)
-		(layer "B.Cu")
-		(net "Net-(U1-OUT)")
-	)
-	(segment
-		(start 91.125002 112.225)
-		(end 86.83 112.225)
-		(width 0.5)
-		(layer "B.Cu")
-		(net "Net-(U1-OUT)")
-	)
 	(zone

Commit message: Fixed diode direction on led-dimmer PCB
Parts:
- turned D1 to -90 degrees
- turned D2 to 90 degrees
Connections:
- D1 pad 1: Net-(D1-K) -> DISCHARGE
- D1 pad 2: DISCHARGE -> Net-(D1-A)
- D2 pad 1: DISCHARGE -> Net-(D2-K)
- D2 pad 2: Net-(D2-A) -> DISCHARGE
- R3 pad 1: Net-(D2-A) -> Net-(D2-K)
- R3 pad 3: Net-(D1-K) -> Net-(D1-A)
Routing:
- net Net-(D1-K): track 3.69 -> 0.00 mm
- net Net-(D1-A): track 0.00 -> 3.69 mm
- net Net-(D2-K): track 0.00 -> 3.65 mm
- net Net-(D2-A): track 3.65 -> 0.00 mm
Other:
- board text added: "LED Dimmer Rev. 1.3"
- board text removed: "LED Dimmer Rev. 1.2"
