File: led-dimmer/led-dimmer.kicad_sch (KiCad schematic)
At the start: 14 parts, among them J1 Conn_01x02_Pin, J2 Conn_01x02_Pin, Q1 IRLML6344, U1 NE555P

Commit message: Updated LED Dimmer PCB decoupling capacitor placement on pin 8
Parts:
- C1, C4, R2, R4: KiLib_Generator (none) -> SMD_2terminal_chip_molded
- C3: KiLib_Generator (none) -> capacitor/THT/other
- Q1: KiLib_Generator (none) -> package/gullwing
- R3: value H50115K1A -> RK09711100F8
- U1: KiLib_Generator (none) -> package/DIP/legacy
Changed lines of the file:
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@@
 	(title_block
 		(title "LED Dimmer Schematic")
-		(date "2026-10-18")
-		(rev "1.3")
+		(date "2026-10-19")
+		(rev "1.4")
 	)
 	(text_box "Power Input"
@@
 			)
 		)
+		(property "KiLib_Generator" "SMD_2terminal_chip_molded"
+			(at 124.46 39.37 0)
+			(hide yes)
+			(show_name no)
+			(do_not_autoplace no)
+			(effects
+				(font
+					(size 1.27 1.27)
+				)
+			)
+		)
 		(pin "1"
 		)
@@
 			)
 		)
+		(property "KiLib_Generator" "SMD_2terminal_chip_molded"
+			(at 30.48 52.07 0)
+			(hide yes)
+			(show_name no)
+			(do_not_autoplace no)
+			(effects
+				(font
+					(size 1.27 1.27)
+				)
+			)
+		)
 		(pin "2"
 		)
@@
 		)
 		(property "Description" "Resistor"
+			(at 72.39 49.53 0)
+			(hide yes)
+			(show_name no)
+			(do_not_autoplace no)
+			(effects
+				(font
+					(size 1.27 1.27)
+				)
+			)
+		)
+		(property "KiLib_Generator" "SMD_2terminal_chip_molded"
 			(at 72.39 49.53 0)
 			(hide yes)
@@
 			)
 		)
+		(property "KiLib_Generator" "capacitor/THT/other"
+			(at 54.61 92.71 0)
+			(hide yes)
+			(show_name no)
+			(do_not_autoplace no)
+			(effects
+				(font
+					(size 1.27 1.27)
+				)
+			)
+		)
 		(pin "1"
 		)
@@
 			)
 		)
+		(property "KiLib_Generator" "SMD_2terminal_chip_molded"
+			(at 63.5 27.94 0)
+			(hide yes)
+			(show_name no)
+			(do_not_autoplace no)
+			(effects
+				(font
+					(size 1.27 1.27)
+				)
+			)
+		)
 		(pin "2"
 		)
@@
 		(fields_autoplaced yes)
 		(property "Reference" "R3"
-			(at 97.7899 46.99 90)
-			(show_name no)
-			(do_not_autoplace no)
-			(effects
-				(font
-					(size 1.27 1.27)
-				)
-				(justify left)
-			)
-		)
-		(property "Value" "H50115K1A"
-			(at 100.3299 46.99 90)
-			(show_name no)
-			(do_not_autoplace no)
-			(effects
-				(font
-					(size 1.27 1.27)
-				)
-				(justify left)
+			(at 99.06 48.26 0)
+			(show_name no)
+			(do_not_autoplace no)
+			(effects
+				(font
+					(size 1.27 1.27)
+				)
+			)
+		)
+		(property "Value" "RK09711100F8"
+			(at 99.06 50.8 0)
+			(show_name no)
+			(do_not_autoplace no)
+			(effects
+				(font
+					(size 1.27 1.27)
+				)
 			)
 		)
@@
 			)
 		)
+		(property "KiLib_Generator" "package/DIP/legacy"
+			(at 57.15 45.72 0)
+			(hide yes)
+			(show_name no)
+			(do_not_autoplace no)
+			(effects
+				(font
+					(size 1.27 1.27)
+				)
+			)
+		)
 		(pin "8"
 		)
@@
 			(at 132.08 44.45 0)
 			(hide yes)
+			(show_name no)
+			(do_not_autoplace no)
+			(effects
+				(font
+					(size 1.27 1.27)
+				)
+			)
+		)
+		(property "KiLib_Generator" "package/gullwing"
+			(at 132.08 44.45 0)
+			(hide yes)

Commit message: LED Dimmer - reorganized project libraries into libs directory
Parts:
- J1, J2: footprint footprints:JST_B2B-XH-A -> external_footprints:JST_B2B-XH-A
- R3: footprint footprints:TRIM_PTN091-H50115K1A -> external_footprints:TRIM_PTN091-H50115K1A
Other:
- company: (none) -> Salinder Sidhu
Changed lines of the file:
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@@
 	(title_block
 		(title "LED Dimmer Schematic")
-		(date "2026-10-19")
+		(date "2026-10-20")
 		(rev "1.4")
+		(company "Salinder Sidhu")
 	)
 	(text_box "Power Input"
@@
 			)
 		)
-		(property "Footprint" "footprints:JST_B2B-XH-A"
+		(property "Footprint" "external_footprints:JST_B2B-XH-A"
 			(at 114.3 91.44 0)
 			(hide yes)
@@
 			)
 		)
-		(property "Footprint" "footprints:TRIM_PTN091-H50115K1A"
+		(property "Footprint" "external_footprints:TRIM_PTN091-H50115K1A"
 			(at 99.06 44.45 0)
 			(hide yes)
@@
 			)
 		)
-		(property "Footprint" "footprints:JST_B2B-XH-A"
+		(property "Footprint" "external_footprints:JST_B2B-XH-A"
 			(at 39.37 87.63 0)
 			(hide yes)
