File: stereo-amplifier-dual-btl-tda2822/stereo-amplifier-dual-btl-tda2822.kicad_sch (KiCad schematic)
At the start: 29 parts, among them J1 SPK L, J2 SPK R, J3 PWR IN, J4 AUX IN, U1 TDA2822, U2 TDA2822

Commit message: Redesign stereo amplifier PCB for Rev 2.0
Parts:
- C1, C2: value 2.2u -> 4.7u
- C10, C11: value 220u -> 470u; footprint Capacitor_THT:CP_Radial_D6.3mm_P2.50mm -> Capacitor_THT:CP_Radial_D8.0mm_P3.50mm
- C3, C4: footprint Capacitor_THT:C_Disc_D3.8mm_W2.6mm_P2.50mm -> Capacitor_SMD:C_0805_2012Metric
- C5, C6: value 10u -> 22u; footprint Capacitor_THT:CP_Radial_D4.0mm_P1.50mm -> Capacitor_THT:CP_Radial_D5.0mm_P2.00mm
- C7, C8: footprint footprints:CAPRR500W50L730T450H950 -> Capacitor_SMD:C_0805_2012Metric
- R1, R2, R3, R4: footprint Resistor_THT:R_Axial_DIN0207_L6.3mm_D2.5mm_P10.16mm_Horizontal -> Resistor_SMD:R_0805_2012Metric_Pad1.20x1.40mm_HandSolder
- R5, R6, R7, R8: footprint Resistor_THT:R_Axial_DIN0207_L6.3mm_D2.5mm_P10.16mm_Horizontal -> Resistor_SMD:R_1206_3216Metric_Pad1.30x1.75mm_HandSolder
Changed lines of the file:
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@@
 	(title_block
 		(title "Stereo Amplifier Dual BTL TDA2822 Schematic")
-		(date "2026-07-01")
-		(rev "1.0")
+		(date "2026-07-08")
+		(rev "2.0")
 		(company "Salinder Sidhu")
 	)
@@
 			)
 		)
-		(property "Footprint" "Resistor_THT:R_Axial_DIN0207_L6.3mm_D2.5mm_P10.16mm_Horizontal"
+		(property "Footprint" "Resistor_SMD:R_1206_3216Metric_Pad1.30x1.75mm_HandSolder"
 			(at 109.728 45.72 90)
 			(hide yes)
@@
 			)
 		)
-		(property "Footprint" "Resistor_THT:R_Axial_DIN0207_L6.3mm_D2.5mm_P10.16mm_Horizontal"
+		(property "Footprint" "Resistor_SMD:R_0805_2012Metric_Pad1.20x1.40mm_HandSolder"
 			(at 28.702 118.11 90)
 			(hide yes)
@@
 			)
 		)
-		(property "Footprint" "footprints:CAPRR500W50L730T450H950"
+		(property "Footprint" "Capacitor_SMD:C_0805_2012Metric"
 			(at 89.2048 114.3 0)
 			(hide yes)
@@
 			)
 		)
-		(property "Footprint" "Capacitor_THT:C_Disc_D3.8mm_W2.6mm_P2.50mm"
+		(property "Footprint" "Capacitor_SMD:C_0805_2012Metric"
 			(at 66.3448 114.3 0)
 			(hide yes)
@@
 			)
 		)
-		(property "Footprint" "Resistor_THT:R_Axial_DIN0207_L6.3mm_D2.5mm_P10.16mm_Horizontal"
+		(property "Footprint" "Resistor_SMD:R_0805_2012Metric_Pad1.20x1.40mm_HandSolder"
 			(at 33.782 43.18 90)
 			(hide yes)
@@
 			)
 		)
-		(property "Footprint" "Resistor_THT:R_Axial_DIN0207_L6.3mm_D2.5mm_P10.16mm_Horizontal"
+		(property "Footprint" "Resistor_SMD:R_0805_2012Metric_Pad1.20x1.40mm_HandSolder"
 			(at 28.702 83.82 90)
 			(hide yes)
@@
 			)
 		)
-		(property "Footprint" "Resistor_THT:R_Axial_DIN0207_L6.3mm_D2.5mm_P10.16mm_Horizontal"
+		(property "Footprint" "Resistor_SMD:R_0805_2012Metric_Pad1.20x1.40mm_HandSolder"
 			(at 65.532 43.18 90)
 			(hide yes)
@@
 			)
 		)
-		(property "Footprint" "footprints:CAPRR500W50L730T450H950"
+		(property "Footprint" "Capacitor_SMD:C_0805_2012Metric"
 			(at 89.2048 80.01 0)
 			(hide yes)
@@
 			)
 		)
-		(property "Footprint" "Resistor_THT:R_Axial_DIN0207_L6.3mm_D2.5mm_P10.16mm_Horizontal"
+		(property "Footprint" "Resistor_SMD:R_1206_3216Metric_Pad1.30x1.75mm_HandSolder"
 			(at 141.478 45.72 90)
 			(hide yes)
@@
 			)
 		)
-		(property "Footprint" "Capacitor_THT:C_Disc_D3.8mm_W2.6mm_P2.50mm"
+		(property "Footprint" "Capacitor_SMD:C_0805_2012Metric"
 			(at 66.3448 80.01 0)
 			(hide yes)
@@
 			)
 		)
-		(property "Value" "10u"
+		(property "Value" "22u"
 			(at 82.55 120.2689 0)
 			(show_name no)
@@
 			)
 		)
-		(property "Footprint" "Capacitor_THT:CP_Radial_D4.0mm_P1.50mm"
+		(property "Footprint" "Capacitor_THT:CP_Radial_D5.0mm_P2.00mm"
 			(at 77.7748 114.3 0)
 			(hide yes)
@@
 			)
 		)
-		(property "Value" "2.2u"
+		(property "Value" "4.7u"
 			(at 41.656 42.164 0)
 			(show_name no)
@@
 			)
 		)
-		(property "Value" "2.2u"
+		(property "Value" "4.7u"
 			(at 54.356 42.164 0)
 			(show_name no)
@@
 			)
 		)
-		(property "Footprint" "Resistor_THT:R_Axial_DIN0207_L6.3mm_D2.5mm_P10.16mm_Horizontal"
+		(property "Footprint" "Resistor_SMD:R_1206_3216Metric_Pad1.30x1.75mm_HandSolder"
 			(at 128.778 45.72 90)
 			(hide yes)
@@
 			)
 		)
-		(property "Value" "220u"
+		(property "Value" "470u"
 			(at 105.41 118.4909 0)
 			(show_name no)
@@
 			)
 		)
-		(property "Footprint" "Capacitor_THT:CP_Radial_D6.3mm_P2.50mm"
+		(property "Footprint" "Capacitor_THT:CP_Radial_D8.0mm_P3.50mm"
 			(at 102.5652 121.92 0)
 			(hide yes)
@@
 			)
 		)
-		(property "Footprint" "Resistor_THT:R_Axial_DIN0207_L6.3mm_D2.5mm_P10.16mm_Horizontal"
+		(property "Footprint" "Resistor_SMD:R_1206_3216Metric_Pad1.30x1.75mm_HandSolder"
 			(at 97.028 45.72 90)
 			(hide yes)
@@
 			)
 		)
-		(property "Value" "220u"
+		(property "Value" "470u"
 			(at 105.41 84.2009 0)
 			(show_name no)
@@
 			)
 		)
-		(property "Footprint" "Capacitor_THT:CP_Radial_D6.3mm_P2.50mm"
+		(property "Footprint" "Capacitor_THT:CP_Radial_D8.0mm_P3.50mm"
 			(at 102.5652 87.63 0)
 			(hide yes)
@@
 			)
 		)
-		(property "Value" "10u"
+		(property "Value" "22u"
 			(at 82.55 85.9789 0)
 			(show_name no)
@@
 			)
 		)
-		(property "Footprint" "Capacitor_THT:CP_Radial_D4.0mm_P1.50mm"
+		(property "Footprint" "Capacitor_THT:CP_Radial_D5.0mm_P2.00mm"
 			(at 77.7748 80.01 0)
 			(hide yes)
