File: stereo-amplifier-dual-btl-tda2822/stereo-amplifier-dual-btl-tda2822.kicad_sch (KiCad schematic)
At the start: 29 parts, among them J1 SPK L, J2 SPK R, J3 PWR IN, J4 AUX IN, U1 TDA2822, U2 TDA2822

Commit message: Stereo Amplifier Dual BTL TDA2822 - reorganized project libraries into libs directory
Parts:
- C12, C13, C14, C9: footprint footprints:CAPRR500W50L730T450H950 -> external_footprints:CAPRR500W50L730T450H950
- J1, J2, J3: footprint footprints:JST_B2B-XH-A -> external_footprints:JST_B2B-XH-A
- J4: footprint footprints:CUI_SJ1-3513N -> external_footprints:CUI_SJ1-3513N
- U1, U2: footprint footprints:DIP762W45P254L1092H508Q8 -> external_footprints:DIP762W45P254L1092H508Q8
Changed lines of the file:
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@@
 	(title_block
 		(title "Stereo Amplifier Dual BTL TDA2822 Schematic")
-		(date "2026-09-09")
+		(date "2026-10-19")
 		(rev "2.1")
 		(company "Salinder Sidhu")
@@
 			)
 		)
-		(property "Footprint" "footprints:JST_B2B-XH-A"
+		(property "Footprint" "external_footprints:JST_B2B-XH-A"
 			(at 135.89 73.66 0)
 			(hide yes)
@@
 			)
 		)
-		(property "Footprint" "footprints:DIP762W45P254L1092H508Q8"
+		(property "Footprint" "external_footprints:DIP762W45P254L1092H508Q8"
 			(at 49.53 77.47 0)
 			(hide yes)
@@
 			)
 		)
-		(property "Footprint" "footprints:CAPRR500W50L730T450H950"
+		(property "Footprint" "external_footprints:CAPRR500W50L730T450H950"
 			(at 126.0348 34.29 0)
 			(hide yes)
@@
 			)
 		)
-		(property "Footprint" "footprints:CAPRR500W50L730T450H950"
+		(property "Footprint" "external_footprints:CAPRR500W50L730T450H950"
 			(at 106.9848 34.29 0)
 			(hide yes)
@@
 			)
 		)
-		(property "Footprint" "footprints:CAPRR500W50L730T450H950"
+		(property "Footprint" "external_footprints:CAPRR500W50L730T450H950"
 			(at 94.2848 34.29 0)
 			(hide yes)
@@
 			)
 		)
-		(property "Footprint" "footprints:CAPRR500W50L730T450H950"
+		(property "Footprint" "external_footprints:CAPRR500W50L730T450H950"
 			(at 138.7348 34.29 0)
 			(hide yes)
@@
 			)
 		)
-		(property "Footprint" "footprints:JST_B2B-XH-A"
+		(property "Footprint" "external_footprints:JST_B2B-XH-A"
 			(at 134.62 25.4 0)
 			(hide yes)
@@
 			)
 		)
-		(property "Footprint" "footprints:DIP762W45P254L1092H508Q8"
+		(property "Footprint" "external_footprints:DIP762W45P254L1092H508Q8"
 			(at 49.53 111.76 0)
 			(hide yes)
@@
 			)
 		)
-		(property "Footprint" "footprints:CUI_SJ1-3513N"
+		(property "Footprint" "external_footprints:CUI_SJ1-3513N"
 			(at 140.97 115.57 0)
 			(hide yes)
@@
 			)
 		)
-		(property "Footprint" "footprints:JST_B2B-XH-A"
+		(property "Footprint" "external_footprints:JST_B2B-XH-A"
 			(at 102.87 25.4 0)
 			(hide yes)
