File: stereo-amplifier-tda2822/stereo-amplifier-tda2822.kicad_pcb (KiCad board)
At the start: 2 copper layers, 50.6 x 54.6 mm, 30 parts, among them J1 PWR IN, J2 AUX IN, J3 SPK 1, J4 SPK 2, U1 TDA2822

Commit message: Update Stereo Amplifier TDA2822 project
Parts:
- removed the C10 at (155.7, 89.9)
- removed the C4 at (138.2, 95.5)
- added C5: 0.1u, footprints:CAPRR500W50L730T450H950, F.Cu at (155.7, 89.9)
- added C7: 100u, Capacitor_THT:CP_Radial_D5.0mm_P2.50mm, F.Cu at (138.2, 95.5)
- added G***: LOGO, footprints:SalSig, B.Cu at (126.0, 113.1)
- added G***: LOGO, footprints:SalLogo, B.Cu at (125.9, 109.8)
- C6: value 100u -> 0.1u; footprint Capacitor_THT:CP_Radial_D5.0mm_P2.50mm -> footprints:CAPRR500W50L730T450H950
- C8: value 0.1u -> 100u; footprint footprints:CAPRR500W50L730T450H950 -> Capacitor_THT:CP_Radial_D5.0mm_P2.50mm
- moved R5 37.4 mm to (164.1, 103.6)
- moved R6 37.4 mm to (126.7, 103.6)
- moved C6 18.4 mm to (135.1, 89.9)
- moved C8 18.4 mm to (152.6, 95.5)
- renumbered C3 to C1, C2 to C10, C5 to C2, C7 to C3, C9 to C4, C1 to C9, J2 to J1, J3 to J2, J4 to J3, J1 to J4, R4 to R2, R2 to R3, R3 to R4
Connections:
- net IN1 + renamed LIN
- net IN2 + renamed RIN
- C6 pad 1: IN1 - -> Net-(C6-Pad1)
- C6 pad 2: GND -> OUT2
- C8 pad 2: OUT2 -> GND
- R5 pad 2: Net-(C8-Pad1) -> Net-(C5-Pad1)
- R6 pad 2: Net-(C10-Pad1) -> Net-(C6-Pad1)
- U1 pad 5: IN2 - -> Net-(C7-Pad1)
- U1 pad 8: IN1 - -> Net-(C8-Pad1)
Routing:
- net Net-(C6-Pad1): track 0.00 -> 7.81 mm
- net Net-(C5-Pad1): track 0.00 -> 7.73 mm
- net Net-(C10-Pad1): track 7.73 -> 0.00 mm
- net Net-(C8-Pad1): track 7.81 -> 3.42 mm
- net IN1 -: track 3.42 -> 0.00 mm
- net Net-(C7-Pad1): track 0.00 -> 3.39 mm
- net IN2 -: track 3.39 -> 0.00 mm
- net GND: vias 51 -> 93
