File: stereo-amplifier-tda2822/stereo-amplifier-tda2822.kicad_pcb (KiCad board)
At the start: 2 copper layers, 50.6 x 54.6 mm, 32 parts, among them J1 AUX IN, J2 SPK 1, J3 SPK 2, J4 PWR IN, U1 TDA2822

Commit message: Stereo Amplifier TDA2822 - reorganized project libraries into libs directory
Parts:
- removed the G*** at (166.3, 110.2)
- removed the G*** at (166.2, 113.5)
- removed the G*** at (126.0, 113.1)
- removed the G*** at (125.9, 109.8)
- added G***: LOGO, sal_footprints:SalLogo, F.Cu at (166.3, 110.2)
- added G***: LOGO, sal_footprints:SalSig, F.Cu at (166.2, 113.5)
- added G***: LOGO, sal_footprints:SalLogo, B.Cu at (125.9, 109.8)
- added G***: LOGO, sal_footprints:SalSig, B.Cu at (126.0, 113.1)
- C10, C5, C6: footprint footprints:CAPRR500W50L730T450H950 -> external_footprints:CAPRR500W50L730T450H950
- J1: footprint footprints:CUI_SJ1-3513N -> external_footprints:CUI_SJ1-3513N
- J2, J3, J4: footprint footprints:JST_B2B-XH-A -> external_footprints:JST_B2B-XH-A
- U1: footprint footprints:DIP762W45P254L1092H508Q8 -> external_footprints:DIP762W45P254L1092H508Q8
