File: stereo-amplifier-tda2822/stereo-amplifier-tda2822.kicad_sch (KiCad schematic)
At the start: 22 parts, among them J1 AUX IN, J2 SPK 1, J3 SPK 2, J4 PWR IN, U1 TDA2822

Commit message: Stereo Amplifier TDA2822 - reorganized project libraries into libs directory
Parts:
- C10, C5, C6: footprint footprints:CAPRR500W50L730T450H950 -> external_footprints:CAPRR500W50L730T450H950
- J1: footprint footprints:CUI_SJ1-3513N -> external_footprints:CUI_SJ1-3513N
- J2, J3, J4: footprint footprints:JST_B2B-XH-A -> external_footprints:JST_B2B-XH-A
- U1: footprint footprints:DIP762W45P254L1092H508Q8 -> external_footprints:DIP762W45P254L1092H508Q8
Changed lines of the file:
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@@
 	(title_block
 		(title "Stereo Amplifier TDA2822 Schematic")
-		(date "2026-08-01")
+		(date "2026-10-19")
 		(rev "3.0")
 		(company "Salinder Sidhu")
@@
 			)
 		)
-		(property "Footprint" "footprints:JST_B2B-XH-A"
+		(property "Footprint" "external_footprints:JST_B2B-XH-A"
 			(at 133.35 82.55 0)
 			(hide yes)
@@
 			)
 		)
-		(property "Footprint" "footprints:CUI_SJ1-3513N"
+		(property "Footprint" "external_footprints:CUI_SJ1-3513N"
 			(at 138.43 127 0)
 			(hide yes)
@@
 			)
 		)
-		(property "Footprint" "footprints:JST_B2B-XH-A"
+		(property "Footprint" "external_footprints:JST_B2B-XH-A"
 			(at 127 26.67 0)
 			(hide yes)
@@
 			)
 		)
-		(property "Footprint" "footprints:CAPRR500W50L730T450H950"
+		(property "Footprint" "external_footprints:CAPRR500W50L730T450H950"
 			(at 86.6648 92.71 0)
 			(hide yes)
@@
 			)
 		)
-		(property "Footprint" "footprints:DIP762W45P254L1092H508Q8"
+		(property "Footprint" "external_footprints:DIP762W45P254L1092H508Q8"
 			(at 52.07 85.09 0)
 			(hide yes)
@@
 			)
 		)
-		(property "Footprint" "footprints:CAPRR500W50L730T450H950"
+		(property "Footprint" "external_footprints:CAPRR500W50L730T450H950"
 			(at 118.4148 43.18 0)
 			(hide yes)
@@
 			)
 		)
-		(property "Footprint" "footprints:JST_B2B-XH-A"
+		(property "Footprint" "external_footprints:JST_B2B-XH-A"
 			(at 104.14 26.67 0)
 			(hide yes)
@@
 			)
 		)
-		(property "Footprint" "footprints:CAPRR500W50L730T450H950"
+		(property "Footprint" "external_footprints:CAPRR500W50L730T450H950"
 			(at 95.5548 43.18 0)
 			(hide yes)
