File: usb-pd-module/usb-pd-module.kicad_pcb (KiCad board)
At the start: 2 copper layers, 34.3 x 46.3 mm, 33 parts, among them J1 USBC, J2 OUT, U1 CH221K, U2 SPX1117M3

Commit message: Updated USB PD Module via placement and increased trace widths of some power paths
Routing:
- net VBUS: track 24.8 -> 26.2 mm, vias 1 -> 2
- net GND: vias 24 -> 55
Other:
- board text added: "USB PD Module Rev. 4.7"
- board text removed: "USB PD Module Rev. 4.6"

Commit message: USB PD Module - reorganized project libraries into libs directory
Parts:
- removed the G*** at (38.4, 53.2)
- removed the G*** at (38.4, 49.9)
- added G***: LOGO, sal_footprints:SalLogo, F.Cu at (38.4, 49.9)
- added G***: LOGO, sal_footprints:SalSig, F.Cu at (38.4, 53.2)
- J1: footprint footprints:AMPHENOL_10164359-00011LF -> external_footprints:AMPHENOL_10164359-00011LF
- J2: footprint footprints:JST_B2B-XH-A -> external_footprints:JST_B2B-XH-A
- S1: footprint footprints:SW_DS04-254-1L-05BK -> external_footprints:SW_DS04-254-1L-05BK
- S2: footprint footprints:SW_100SP1T2B4M7QE -> external_footprints:SW_100SP1T2B4M7QE
