File: usb-pd-module/usb-pd-module.kicad_sch (KiCad schematic)
At the start: 25 parts, among them J1 USBC, J2 OUT, U1 CH221K, U2 SPX1117M3

Commit message: USB PD Module - reorganized project libraries into libs directory
Parts:
- J1: footprint footprints:AMPHENOL_10164359-00011LF -> external_footprints:AMPHENOL_10164359-00011LF
- J2: footprint footprints:JST_B2B-XH-A -> external_footprints:JST_B2B-XH-A
- S1: footprint footprints:SW_DS04-254-1L-05BK -> external_footprints:SW_DS04-254-1L-05BK
- S2: footprint footprints:SW_100SP1T2B4M7QE -> external_footprints:SW_100SP1T2B4M7QE
Changed lines of the file:
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@@
 	(title_block
 		(title "USB PD Module Schematic")
-		(date "2026-09-08")
+		(date "2026-10-19")
 		(rev "4.7")
 		(company "Salinder Sidhu")
@@
 			)
 		)
-		(property "Footprint" "footprints:AMPHENOL_10164359-00011LF"
+		(property "Footprint" "external_footprints:AMPHENOL_10164359-00011LF"
 			(at 45.72 44.45 0)
 			(hide yes)
@@
 			)
 		)
-		(property "Footprint" "footprints:JST_B2B-XH-A"
+		(property "Footprint" "external_footprints:JST_B2B-XH-A"
 			(at 170.18 97.79 0)
 			(hide yes)
@@
 			)
 		)
-		(property "Footprint" "footprints:SW_100SP1T2B4M7QE"
+		(property "Footprint" "external_footprints:SW_100SP1T2B4M7QE"
 			(at 46.99 66.04 0)
 			(hide yes)
@@
 			)
 		)
-		(property "Footprint" "footprints:SW_DS04-254-1L-05BK"
+		(property "Footprint" "external_footprints:SW_DS04-254-1L-05BK"
 			(at 41.91 113.03 0)
 			(hide yes)
